Commit message: change the code

File: model/gazebo_env_setup.xacro (robot description, xacro)
@@ -12,5 +12,5 @@
     </xacro:include>
     <joint name="table_fixed_1" type="fixed">
-      <origin rpy="0 0 0" xyz="0.6 0.0 0.0"/>
+      <origin rpy="0 0 0" xyz="0.68 0.0 0.0"/>
       <parent link="world"/>
       <child link="table_front"/>
