Commit message: move models from birl_baxter_describtion to this repo

File: model/container.xacro (robot description, xacro)
@@ -5,5 +5,5 @@
       <origin rpy="0 0 0" xyz="0 0 0"/>
       <geometry>
-        <mesh filename="package://birl_baxter_description/meshes/container/container.STL"/>
+        <mesh filename="package://birl_kitting_experiment_simulation/meshes/container/container.STL"/>
       </geometry>
     </visual>
@@ -11,5 +11,5 @@
       <origin rpy="0 0 0" xyz="0 0 0"/>
       <geometry>
-        <mesh filename="package://birl_baxter_description/meshes/container/container.STL"/>
+        <mesh filename="package://birl_kitting_experiment_simulation/meshes/container/container.STL"/>
       </geometry>
     </collision>

File: model/table_front.xacro (robot description, xacro)
@@ -5,5 +5,5 @@
       <origin rpy="0 0 0" xyz="0 0 0"/>
       <geometry>
-        <mesh filename="package://birl_baxter_description/meshes/table/table.dae"/>
+        <mesh filename="package://birl_kitting_experiment_simulation/meshes/table/table.dae"/>
       </geometry>
     </visual>
@@ -11,5 +11,5 @@
       <origin rpy="0 0 0" xyz="0 0 0"/>
       <geometry>
-        <mesh filename="package://birl_baxter_description/meshes/table/table.stl"/>
+        <mesh filename="package://birl_kitting_experiment_simulation/meshes/table/table.stl"/>
       </geometry>
     </collision>

File: model/table_right_side.xacro (robot description, xacro)
@@ -5,5 +5,5 @@
       <origin rpy="0 0 0" xyz="0.0 -0.2 0"/>
       <geometry>
-        <mesh filename="package://birl_baxter_description/meshes/table/table.dae"/>
+        <mesh filename="package://birl_kitting_experiment_simulation/meshes/table/table.dae"/>
       </geometry>
     </visual>
@@ -11,5 +11,5 @@
       <origin rpy="0 0 0" xyz="0.0 -0.2 0"/>
       <geometry>
-        <mesh filename="package://birl_baxter_description/meshes/table/table.stl"/>
+        <mesh filename="package://birl_kitting_experiment_simulation/meshes/table/table.stl"/>
       </geometry>
     </collision>
